File: RicardoTemplate.kicad_pcb (KiCad board)
At the start: 4 copper layers, 16 parts, among them U3 LM66200DRLR, U4 MAX77827AEFD+T, U5 SC4215ASTRT

Commit message: Alpha revision
Bulk of routing, layout and etc... is done, design needs to be refined, via stitched and reviewed.
Parts:
- added 12VLED1: RED_LED, Resistor_SMD:R_0402_1005Metric, F.Cu at (145.5, 89.2)
- added 3V3LED1: BLUE_LED, Resistor_SMD:R_0402_1005Metric, F.Cu at (161.2, 85.8)
- added ?: , , F.Cu at (162.3, 125.0)
- added ANT1: TestPoint, TestPoint:TestPoint_Pad_D1.0mm, F.Cu at (163.6, 109.3)
- added BOOTJUMPER1: Conn_01x02_Male, Connector_PinHeader_2.54mm:PinHeader_1x02_P2.54mm_Vertical, F.Cu at (140.7, 120.1)
- added BOOTJUMPER2: Conn_01x02_Male, Connector_PinHeader_2.54mm:PinHeader_1x02_P2.54mm_Vertical, F.Cu at (172.1, 106.9)
- added BOOTJUMPER3: Conn_01x02_Male, Connector_PinHeader_2.54mm:PinHeader_1x02_P2.54mm_Vertical, F.Cu at (143.0, 94.9)
- added BUSY1: TestPoint, TestPoint:TestPoint_Pad_D1.0mm, F.Cu at (159.1, 111.5)
- added C1: 10uF, Capacitor_SMD:C_0402_1005Metric, F.Cu at (154.4, 108.7)
- added C10: 0.1uF, Capacitor_SMD:C_0402_1005Metric, F.Cu at (151.6, 96.6)
- added C11: 0.1uF, Capacitor_SMD:C_0402_1005Metric, F.Cu at (162.1, 101.7)
- added C13: 11pF, Capacitor_SMD:C_0402_1005Metric, F.Cu at (149.5, 100.2)
- added C14: 11pF, Capacitor_SMD:C_0402_1005Metric, F.Cu at (149.5, 104.1)
- added C15: 100nF, Capacitor_SMD:C_0402_1005Metric, F.Cu at (159.0, 85.8)
- added C16: 10uF, Capacitor_SMD:C_0402_1005Metric, F.Cu at (157.8, 85.8)
- added C17: 47nF, Capacitor_SMD:C_0402_1005Metric, F.Cu at (151.8, 81.0)
- added C2: 1uF, Capacitor_SMD:C_0402_1005Metric, F.Cu at (155.9, 107.3)
- added C3: 0.1uF, Capacitor_SMD:C_0402_1005Metric, F.Cu at (139.4, 112.9)
- added C4: 1uF, Capacitor_SMD:C_0402_1005Metric, F.Cu at (154.4, 109.8)
- added C5: 0.1uF, Capacitor_SMD:C_0402_1005Metric, F.Cu at (154.4, 107.7)
- added C50: C_Small, Capacitor_SMD:C_0402_1005Metric, F.Cu at (161.5, 115.1)
- added C51: C_Small, Capacitor_SMD:C_0402_1005Metric, F.Cu at (158.7, 115.0)
- added C52: 10nF, Capacitor_SMD:C_0402_1005Metric, F.Cu at (163.5, 116.6)
- added C53: 10nF, Capacitor_SMD:C_0402_1005Metric, F.Cu at (163.2, 117.7)
- added C54: 0.1uF, Capacitor_SMD:C_0402_1005Metric, F.Cu at (157.6, 121.4)
- added C57: 470nF, Capacitor_SMD:C_0402_1005Metric, F.Cu at (157.7, 122.4)
- added C58: 0.1uF, Capacitor_SMD:C_0402_1005Metric, F.Cu at (161.1, 125.1)
- added C59: 1nF, Capacitor_SMD:C_0402_1005Metric, F.Cu at (171.3, 124.1)
- added C6: 0.1uF, Capacitor_SMD:C_0402_1005Metric, F.Cu at (154.9, 106.3)
- added C60: 1nF, Capacitor_SMD:C_0402_1005Metric, F.Cu at (172.3, 124.1)
- added C61: 100nF, Capacitor_SMD:C_0402_1005Metric, F.Cu at (177.0, 117.4)
- added C62: 10uF, Capacitor_SMD:C_0402_1005Metric, F.Cu at (185.0, 92.8)
- added C63: 1nF, Capacitor_SMD:C_0402_1005Metric, F.Cu at (173.3, 124.1)
- added C64: 0.1uF, Capacitor_SMD:C_0402_1005Metric, F.Cu at (185.0, 93.8)
- added C65: 1nF, Capacitor_SMD:C_0402_1005Metric, F.Cu at (176.0, 118.3)
- added C66: 1nF, Capacitor_SMD:C_0402_1005Metric, F.Cu at (171.9, 117.5)
- added C67: 1nF, Capacitor_SMD:C_0402_1005Metric, F.Cu at (172.9, 116.6)
- added C68: 100nF, Capacitor_SMD:C_0402_1005Metric, F.Cu at (170.9, 116.5)
- added C69: 100nF, Capacitor_SMD:C_0402_1005Metric, F.Cu at (168.9, 117.5)
- added C7: 1uF, Capacitor_SMD:C_0402_1005Metric, F.Cu at (152.3, 105.7)
- added C70: 1nF, Capacitor_SMD:C_0402_1005Metric, F.Cu at (174.5, 118.0)
- added C71: 4.7uF, Capacitor_SMD:C_0603_1608Metric, F.Cu at (169.6, 115.0)
- added C72: 100nF, Capacitor_SMD:C_0402_1005Metric, F.Cu at (169.9, 117.5)
- added C73: 100nF, Capacitor_SMD:C_0402_1005Metric, F.Cu at (174.5, 117.0)
- added C74: 4.7uF, Capacitor_SMD:C_0603_1608Metric, F.Cu at (174.2, 114.9)
- added C8: 0.1uF, Capacitor_SMD:C_0402_1005Metric, F.Cu at (135.1, 119.6)
- added C9: 10nF, Capacitor_SMD:C_0402_1005Metric, F.Cu at (152.3, 106.7)
- added CHL1: TestPoint, TestPoint:TestPoint_Pad_D1.0mm, F.Cu at (168.2, 105.0)
- added CPS1: TestPoint, TestPoint:TestPoint_Pad_D1.0mm, F.Cu at (170.9, 101.7)
- added CRX1: TestPoint, TestPoint:TestPoint_Pad_D1.0mm, F.Cu at (166.7, 106.6)
- added CRXLED1: ORANGE_LED, Resistor_SMD:R_0402_1005Metric, F.Cu at (155.4, 88.9)
- added CS1: TestPoint, TestPoint:TestPoint_Pad_D1.0mm, F.Cu at (161.1, 94.0)
- added CSD1: TestPoint, TestPoint:TestPoint_Pad_D1.0mm, F.Cu at (165.1, 108.0)
- added CTX1: TestPoint, TestPoint:TestPoint_Pad_D1.0mm, F.Cu at (169.5, 103.3)
- added CTXLED1: GREEN_LED, Resistor_SMD:R_0402_1005Metric, F.Cu at (148.1, 88.7)
- added D1: SM712_SOT23, Package_TO_SOT_SMD:SOT-23, F.Cu at (151.8, 77.9)
- added D2: SP0503BAHT, Package_TO_SOT_SMD:SOT-143, F.Cu at (172.8, 83.1)
- added DIO1: TestPoint, TestPoint:TestPoint_Pad_D1.0mm, F.Cu at (155.2, 112.0)
- added ENJUMPER1: Conn_01x02_Male, Connector_PinHeader_2.54mm:PinHeader_1x02_P2.54mm_Vertical, F.Cu at (140.7, 116.4)
- added FB1: FerriteBead_Small, Inductor_SMD:L_0603_1608Metric, F.Cu at (145.9, 95.7)
- added FB4: FerriteBead_Small, Inductor_SMD:L_0603_1608Metric, F.Cu at (171.9, 113.8)
- added H1: MountingHole_Pad, MountingHole:MountingHole_3.2mm_M3_DIN965_Pad, F.Cu at (123.1, 75.6)
- added H2: MountingHole_Pad, MountingHole:MountingHole_3.2mm_M3_DIN965_Pad, F.Cu at (195.9, 75.6)
- added H3: MountingHole_Pad, MountingHole:MountingHole_3.2mm_M3_DIN965_Pad, F.Cu at (123.1, 130.6)
- added H4: MountingHole_Pad, MountingHole:MountingHole_3.2mm_M3_DIN965_Pad, F.Cu at (195.9, 130.6)
- added IC2: SX1280, footprints:QFN50P400X400X95-24N, F.Cu at (161.4, 120.9)
- added J1: RBUS, Connector_Molex:Molex_Mini-Fit_Jr_5566-06A_2x03_P4.20mm_Vertical, F.Cu at (139.8, 84.0)
- added J2: USB_C_Receptacle_USB2.0, Connector_USB:USB_C_Receptacle_Palconn_UTC16-G, F.Cu at (173.4, 76.4)
- added J4: SMA, Connector_Coaxial:SMA_Amphenol_901-144_Vertical, F.Cu at (185.7, 121.1)
- added JP1: TermJP, Jumper:SolderJumper-2_P1.3mm_Open_RoundedPad1.0x1.5mm, F.Cu at (155.9, 84.0)
- added JTAG1: JTAG, Connector_PinHeader_2.54mm:PinHeader_1x04_P2.54mm_Vertical, F.Cu at (137.6, 125.1)
- added L1: 2.0nH, Inductor_SMD:L_0402_1005Metric, F.Cu at (153.9, 106.3)
- added L2: 20nH, Inductor_SMD:L_0402_1005Metric, F.Cu at (151.8, 102.9)
- added L4: 15uF, Capacitor_SMD:C_0603_1608Metric, F.Cu at (158.9, 124.6)
- added MISO1: TestPoint, TestPoint:TestPoint_Pad_D1.0mm, F.Cu at (154.8, 94.0)
- added MOSI1: TestPoint, TestPoint:TestPoint_Pad_D1.0mm, F.Cu at (156.9, 94.0)
- added R1: 10K, Resistor_SMD:R_0402_1005Metric, F.Cu at (155.9, 109.2)
- added R10: 60, Resistor_SMD:R_0603_1608Metric, F.Cu at (153.9, 81.0)
- added R11: 5.1k, Resistor_SMD:R_0402_1005Metric, F.Cu at (179.3, 76.2)
- added R12: 5.1k, Resistor_SMD:R_0402_1005Metric, F.Cu at (167.2, 76.0)
- added R13: 5.1k, Resistor_SMD:R_0402_1005Metric, F.Cu at (137.4, 90.4)
- added R18: 1k, Resistor_SMD:R_0402_1005Metric, F.Cu at (156.4, 88.9)
- added R2: 470, Resistor_SMD:R_0402_1005Metric, F.Cu at (148.4, 128.4)
- added R24: 1k, Resistor_SMD:R_0402_1005Metric, F.Cu at (163.8, 115.5)
- added R27: 56k, Resistor_SMD:R_0402_1005Metric, F.Cu at (185.0, 91.7)
- added R28: 10k, Resistor_SMD:R_0402_1005Metric, F.Cu at (187.0, 91.7)
- added R3: 10K, Resistor_SMD:R_0402_1005Metric, F.Cu at (157.1, 107.3)
- added R4: 470, Resistor_SMD:R_0402_1005Metric, F.Cu at (160.2, 85.8)
- added R5: 1k, Resistor_SMD:R_0402_1005Metric, F.Cu at (147.1, 88.7)
- added R6: 499R, Resistor_SMD:R_0402_1005Metric, F.Cu at (144.8, 119.9)
- added R7: 3k, Resistor_SMD:R_0402_1005Metric, F.Cu at (145.5, 88.2)
- added R8: 0, Resistor_SMD:R_0603_1608Metric, F.Cu at (148.2, 84.0)
- added R9: 60, Resistor_SMD:R_0603_1608Metric, F.Cu at (149.7, 81.0)
- added RF_RST1: TestPoint, TestPoint:TestPoint_Pad_D1.0mm, F.Cu at (162.0, 110.8)
- added SCK1: TestPoint, TestPoint:TestPoint_Pad_D1.0mm, F.Cu at (159.0, 94.0)
- added TP1: TestPoint, TestPoint:TestPoint_Pad_D1.0mm, F.Cu at (174.1, 86.0)
- added TP10: TestPoint, TestPoint:TestPoint_Pad_D1.0mm, F.Cu at (152.7, 90.7)
- added TP2: TestPoint, TestPoint:TestPoint_Pad_D1.0mm, F.Cu at (171.9, 86.0)
- added TP22: TestPoint, TestPoint:TestPoint_Pad_D1.0mm, F.Cu at (211.7, 117.3)
- added TP23: TestPoint, TestPoint:TestPoint_Pad_D1.0mm, F.Cu at (173.9, 112.1)
- added TP24: TestPoint, TestPoint:TestPoint_Pad_D1.0mm, F.Cu at (206.7, 117.3)
- added TP25: TestPoint, TestPoint:TestPoint_Pad_D1.0mm, F.Cu at (206.7, 120.3)
- added TP4: TestPoint, TestPoint:TestPoint_Pad_D1.5mm, F.Cu at (125.7, 91.3)
- added TP5: TestPoint, TestPoint:TestPoint_Pad_D1.5mm, F.Cu at (127.0, 88.2)
- added TP6: TestPoint, TestPoint:TestPoint_Pad_D1.5mm, F.Cu at (143.4, 98.2)
- added TP8: TestPoint, TestPoint:TestPoint_Pad_D1.5mm, F.Cu at (134.6, 89.0)
- added TP9: TestPoint, TestPoint:TestPoint_Pad_D1.0mm, F.Cu at (150.6, 90.7)
- added TXLED1: GREEN_LED, Resistor_SMD:R_0402_1005Metric, F.Cu at (147.4, 128.4)
- added U1: ESP32-S3, footprints:QFN40P700X700X90-57N, F.Cu at (156.9, 101.1)
- added U11: SC4215ASTRT, footprints:SOIC127P599X175-9N, F.Cu at (185.1, 87.2)
- added U12: SKY66112-11, footprints:SKY66112-11_SKY, F.Cu at (172.8, 120.4)
- added U13: DEA202450BT-1213C1, footprints:DEA-4_2P0X1P25, F.Cu at (178.4, 121.1)
- added U2: SN65HVD230, Package_SO:SOIC-8_3.9x4.9mm_P1.27mm, F.Cu at (151.8, 85.7)
- added UART1: UART, Connector_PinHeader_2.54mm:PinHeader_1x04_P2.54mm_Vertical, F.Cu at (141.4, 125.1)
- added USBLED1: WHITE_LED, Resistor_SMD:R_0402_1005Metric, F.Cu at (138.5, 90.4)
- added Y1: R940000171, Crystal:Crystal_SMD_2016-4Pin_2.0x1.6mm, F.Cu at (149.5, 102.2)
- added Y3: Crystal_GND24, Crystal:Crystal_SMD_2016-4Pin_2.0x1.6mm, F.Cu at (160.1, 116.3)
- U3: footprint iclr:SOTFL50P160X60-8N -> footprints:SOTFL50P160X60-8N
- U4: footprint iclr:CONV_MAX77827AEFD+T -> footprints:CONV_MAX77827AEFD+T
- U5: footprint iclr:SOIC127P599X175-9N -> footprints:SOIC127P599X175-9N
- moved C24 54.9 mm to (128.4, 101.8), turned to 90 degrees
- moved C25 53.7 mm to (128.4, 103.9), turned to -90 degrees
- moved U5 48.9 mm to (132.5, 102.9), turned to 0 degrees
- moved C23 46.8 mm to (129.6, 97.1), turned to 180 degrees
- moved L3 46.1 mm to (127.0, 94.6), turned to -90 degrees
- moved R17 45.1 mm to (136.7, 101.1), turned to 90 degrees
- moved R16 43.7 mm to (136.7, 103.0), turned to 90 degrees
- moved U4 42.9 mm to (130.8, 94.6), turned to 180 degrees
- moved C26 42.5 mm to (136.7, 104.8), turned to 90 degrees
- moved C27 41.3 mm to (137.6, 104.8), turned to 90 degrees
- moved C21 41.2 mm to (129.4, 92.0), turned to 180 degrees
- moved R15 40.9 mm to (133.0, 94.4), turned to 90 degrees
- moved R14 40.3 mm to (128.6, 90.5), turned to 0 degrees
- moved C22 39.1 mm to (132.2, 92.3), turned to 0 degrees
- moved C20 38.0 mm to (132.2, 91.4), turned to 0 degrees
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Connections:
- net +3V3 renamed Net-(BOOTJUMPER3-Pin_2)
- C23 pad 1: /Power/BBOUT -> VBUS
- C24 pad 1: /Power/BBOUT -> VBUS
- C25 pad 1: /Power/BBOUT -> VBUS
- U4 pad 11: /Power/BBOUT -> VBUS
- U4 pad 13: /Power/BBOUT -> VBUS
- U5 pad 2: /Power/BBOUT -> VBUS
- U5 pad 3: /Power/BBOUT -> VBUS
Routing:
- net GND: track 7.31 -> 131.4 mm, vias 8 -> 207
- net VBUS: track 5.51 -> 97.6 mm, vias 2 -> 4
- net CS: track 0.00 -> 40.9 mm, vias 0 -> 2
- net Net-(JTAG1-Pin_4): track 0.00 -> 39.0 mm, vias 0 -> 1
- net SCK: track 0.00 -> 38.0 mm, vias 0 -> 2
- net ANT_SEL: track 0.00 -> 38.0 mm, vias 0 -> 2
- net MISO: track 0.00 -> 37.3 mm, vias 0 -> 2
- net MOSI: track 0.00 -> 37.0 mm, vias 0 -> 2
- net /BOOT: track 0.00 -> 36.5 mm, vias 0 -> 2
- net Net-(JTAG1-Pin_3): track 0.00 -> 36.5 mm, vias 0 -> 1
- net Net-(JTAG1-Pin_1): track 0.00 -> 36.2 mm, vias 0 -> 1
- net Net-(JTAG1-Pin_2): track 0.00 -> 35.1 mm, vias 0 -> 1
- net CSD: track 0.00 -> 34.7 mm, vias 0 -> 2
- net /Data+: track 0.00 -> 34.4 mm, vias 0 -> 2
- net /Data-: track 0.00 -> 34.1 mm, vias 0 -> 2
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- added copper zone on B.Cu, net GND
- added copper zone on In1.Cu, net GND
- added copper zone on F.Cu, net VBUS
- removed copper zone on F.Cu, net /Power/BBOUT
- removed copper zone on F.Cu, net Net-(BOOTJUMPER3-Pin_2)
Other:
- board outline added: 80.2 x 62.6 mm
- board text added: "3V3 NC!"
- board text added: "GND"
- board text added: "MTCK"
- board text added: "MTDI"
- board text added: "MTDO"
- board text added: "MTMS"
- board text added: "RX"
- board text added: "TX"
