File: RicardoTemplate.kicad_pcb (KiCad board)
At the start: 4 copper layers, 80.2 x 62.6 mm, 133 parts, among them IC2 SX1280, J1 RBUS, J2 USB_C_Receptacle_USB2.0, J4 SMA, U1 ESP32-S3, U11 SC4215ASTRT, U12 SKY66112-11, U13 DEA202450BT-1213C1, U2 SN65HVD230, U3 LM66200DRLR, U4 MAX77827AEFD+T, U5 SC4215ASTRT, Y1 R940000171, Y3 Crystal_GND24

Commit message: Minor improvements
Parts:
- removed JTAG1: JTAG, Connector_PinHeader_2.54mm:PinHeader_1x04_P2.54mm_Vertical
- removed TP22, TP24, TP25: TestPoint, TestPoint:TestPoint_Pad_D1.0mm
- renumbered J4 to ANT1, ANT1 to ANT_S1, TP10 to CANRX1, TP9 to CANTX1, FB1 to FB_P1, FB4 to FB_R1, BOOTJUMPER3 to POWER_MAIN1, BOOTJUMPER2 to POWER_RADIO1
Connections:
- C23 pad 1: VBUS -> /Power/BBOUT
- C24 pad 1: VBUS -> /Power/BBOUT
- C25 pad 1: VBUS -> /Power/BBOUT
- TP8 pad 1: VBUS -> /Power/BBOUT
- U1 pad 44: Net-(JTAG1-Pin_4) -> unconnected-(U1-MTCK/JTAG/GPIO39-Pad44)
- U1 pad 45: Net-(JTAG1-Pin_3) -> unconnected-(U1-MTDO/JTAG/GPIO40-Pad45)
- U1 pad 47: Net-(JTAG1-Pin_2) -> unconnected-(U1-MTDI/JTAG/GPIO41-Pad47)
- U1 pad 48: Net-(JTAG1-Pin_1) -> unconnected-(U1-MTMS/JTAG/GPIO42-Pad48)
- U4 pad 11: VBUS -> /Power/BBOUT
- U4 pad 13: VBUS -> /Power/BBOUT
- U5 pad 2: VBUS -> /Power/BBOUT
- U5 pad 3: VBUS -> /Power/BBOUT
Routing:
- net Net-(JTAG1-Pin_4): track 39.0 -> 0.00 mm, vias 1 -> 0
- net Net-(JTAG1-Pin_3): track 36.5 -> 0.00 mm, vias 1 -> 0
- net Net-(JTAG1-Pin_1): track 36.2 -> 0.00 mm, vias 1 -> 0
- net Net-(JTAG1-Pin_2): track 35.1 -> 0.00 mm, vias 1 -> 0
- net VBUS: track 97.6 -> 86.9 mm
- net /Power/BBOUT: track 0.00 -> 1.27 mm
Other:
- board text removed: "MTCK"
- board text removed: "MTDI"
- board text removed: "MTDO"
- board text removed: "MTMS"
