File: RF_Frontend.kicad_sch (KiCad schematic)
At the start: 40 parts, among them IC2 SX1280, J4 SMA, U10 SC4215ASTRT, U11 SC4215ASTRT, U12 SKY66112-11, U13 DEA202450BT-1213C1, Y3 Crystal_GND24

Commit message: Alpha revision
Bulk of routing, layout and etc... is done, design needs to be refined, via stitched and reviewed.
Parts:
- removed C55: 10uF, Capacitor_SMD:C_0402_1005Metric, symbol Device:C_Small
- removed C56: 0.1uF, Capacitor_SMD:C_0402_1005Metric, symbol Device:C_Small
- removed FB3: FerriteBead_Small, symbol Device:FerriteBead_Small
- removed R25: 56k, Resistor_SMD:R_0402_1005Metric, symbol Device:R_Small
- removed R26: 10k, Resistor_SMD:R_0402_1005Metric, symbol Device:R_Small
- removed U10: SC4215ASTRT, iclr:SOIC127P599X175-9N, symbol iclr:SC4215ASTRT
- added ANT1, BUSY1, CHL1, CPS1, CRX1, CS1, CSD1, CTX1, DIO1, MISO1, MOSI1, RF_RST1, SCK1, TP22, TP23: TestPoint, TestPoint:TestPoint_Pad_D1.0mm, symbol Connector:TestPoint
- added BOOTJUMPER2: Conn_01x02_Male, Connector_PinHeader_2.54mm:PinHeader_1x02_P2.54mm_Vertical, symbol Connector:Conn_01x02_Male
- C50, C51, C52, C53, C54, C57, C58, C59, C60, C61, C63, C65, C66, C67, C68, C69, C70, C72, C73: footprint (none) -> Capacitor_SMD:C_0402_1005Metric
- C71, C74, L4: footprint (none) -> Capacitor_SMD:C_0603_1608Metric
- FB4: footprint (none) -> Inductor_SMD:L_0603_1608Metric
- IC2: footprint QFN50P400X400X80-25N-D -> footprints:QFN50P400X400X95-24N
- J4: footprint (none) -> Connector_Coaxial:SMA_Amphenol_901-144_Vertical
- R24: footprint (none) -> Resistor_SMD:R_0402_1005Metric
- U11: footprint iclr:SOIC127P599X175-9N -> footprints:SOIC127P599X175-9N
- U12: footprint SKY66112-11_SKY -> footprints:SKY66112-11_SKY
- U13: footprint DEA-4_2P0X1P25 -> footprints:DEA-4_2P0X1P25
- Y3: footprint (none) -> Crystal:Crystal_SMD_2016-4Pin_2.0x1.6mm
Connections:
- net ANT_SEL: now also ANT1.1
- net CHL: now also CHL1.1
- net CPS: now also CPS1.1; no longer IC2.10 (DIO3)
- net CRX: now also CRX1.1; no longer IC2.8 (DIO1)
- net CS: now also CS1.1
- net CSD: now also CSD1.1
- net CTX: now also CTX1.1; no longer IC2.9 (DIO2)
- net GND: now also C59.2, C60.2, C61.2, C63.2, C65.2, C66.2, C67.2, C68.2, C69.1, C70.2, C71.2, C72.1, C73.2, C74.2, J4.2 (Ext), U12.1 (GND), U12.10 (GND), U12.12 (GND), U12.13 (GND), U12.18 (GND), U12.20 (GND), U12.22 (GND), U12.23 (GND), U12.24 (GND), U12.5 (GND), U12.7 (GND), U12.9 (GND), U13.2 (GND), U13.4 (GND)
- net MISO: now also MISO1.1
- net MOSI: now also MOSI1.1
- net SCK: now also SCK1.1
- net SX_BUSY: now also BUSY1.1
- net VAA: now also C58.1, IC2.15 (VBAT), TP22.1, TP23.1
- net VS: no longer C58.1, IC2.15 (VBAT)
- net at C62.2, C64.2, R27.1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: now also BOOTJUMPER2.2 (Pin_2); no longer FB4.1
- net RF_RST: now reaches R24.1
- net RF_RST: now also RF_RST1.1
- removed net GNDA: C59.2, C60.2, C61.2, C63.2, C65.2, C66.2, C67.2, C68.2, C69.1, C70.2, C71.2, C72.1, C73.2, C74.2, J4.1 (In), J4.2 (Ext), U12.1 (GND), U12.10 (GND), U12.12 (GND), U12.13 (GND), U12.18 (GND), U12.20 (GND), U12.22 (GND), U12.23 (GND), U12.24 (GND), U12.5 (GND), U12.7 (GND), U12.9 (GND), U13.2 (GND), U13.3 (OUT), U13.4 (GND)
- new net: BOOTJUMPER2.1 (Pin_1), FB4.1
- new net: J4.1 (In), U13.3 (OUT)
- new net DIO1: DIO1.1, IC2.8 (DIO1)
- no-connect marks 4 -> 5
Other:
- note added: "Splitting grounds is a dumb idea 99.98% of the time."
- moved on the sheet: C50, C51, C52, C53, C54, C57, C58, C62, C64, FB4, IC2, L4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

Commit message: Minor improvements
Parts:
- removed TP22: TestPoint, TestPoint:TestPoint_Pad_D1.0mm, symbol Connector:TestPoint
- renumbered J4 to ANT1, ANT1 to ANT_S1, FB4 to FB_R1, BOOTJUMPER2 to POWER_RADIO1
Changed lines of the file:
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@@
 	)
 	(junction
-		(at 246.38 36.83)
-		(diameter 0)
-		(color 0 0 0 0)
-	)
-	(junction
 		(at 167.64 83.82)
 		(diameter 0)
@@
 		(on_board yes)
 		(dnp no)
-		(property "Reference" "BOOTJUMPER2"
+		(property "Reference" "POWER_RADIO1"
 			(at 213.36 26.67 90)
 			(effects
@@
 			(project "RicardoTemplate"
 				(path "/7db990e4-92e1-4f99-b4d2-435bbec1ba83/ecfc1314-a0cb-4bac-a35c-d2175f1c7197"
-					(reference "BOOTJUMPER2")
+					(reference "POWER_RADIO1")
 					(unit 1)
 				)
@@
 		(dnp no)
 		(fields_autoplaced yes)
-		(property "Reference" "J4"
-			(at 255.27 141.2631 0)
+		(property "Reference" "ANT1"
+			(at 254 141.2631 0)
 			(effects
 				(font
@@
 		)
 		(property "Value" "SMA"
-			(at 255.27 143.8031 0)
+			(at 254 143.8031 0)
 			(effects
 				(font
@@
 			(project "RicardoTemplate"
 				(path "/7db990e4-92e1-4f99-b4d2-435bbec1ba83/ecfc1314-a0cb-4bac-a35c-d2175f1c7197"
-					(reference "J4")
+					(reference "ANT1")
 					(unit 1)
 				)
@@
 	)
 	(symbol
-		(lib_id "Connector:TestPoint")
-		(at 246.38 36.83 270)
-		(unit 1)
-		(exclude_from_sim no)
-		(in_bom yes)
-		(on_board yes)
-		(dnp no)
-		(property "Reference" "TP22"
-			(at 251.1552 35.6616 90)
-			(effects
-				(font
-					(size 1.27 1.27)
-				)
-				(justify left)
-			)
-		)
-		(property "Value" "TestPoint"
-			(at 251.1552 37.973 90)
-			(effects
-				(font
-					(size 1.27 1.27)
-				)
-				(justify left)
-			)
-		)
-		(property "Footprint" "TestPoint:TestPoint_Pad_D1.0mm"
-			(at 246.38 41.91 0)
-			(effects
-				(font
-					(size 1.27 1.27)
-				)
-				(hide yes)
-			)
-		)
-		(property "Datasheet" "~"
-			(at 246.38 41.91 0)
-			(effects
-				(font
-					(size 1.27 1.27)
-				)
-				(hide yes)
-			)
-		)
-		(property "Description" ""
-			(at 246.38 36.83 0)
-			(effects
-				(font
-					(size 1.27 1.27)
-				)
-				(hide yes)
-			)
-		)
-		(pin "1"
-		)
-		(instances
-			(project "RicardoTemplate"
-				(path "/7db990e4-92e1-4f99-b4d2-435bbec1ba83/ecfc1314-a0cb-4bac-a35c-d2175f1c7197"
-					(reference "TP22")
-					(unit 1)
-				)
-			)
-		)
-	)
-	(symbol
 		(lib_id "Device:C_Small")
 		(at 167.64 87.63 0)
@@
 		(on_board yes)
 		(dnp no)
-		(property "Reference" "ANT1"
+		(property "Reference" "ANT_S1"
 			(at 37.1348 126.8984 90)
 			(effects
@@
 			(project "RicardoTemplate"
 				(path "/7db990e4-92e1-4f99-b4d2-435bbec1ba83/ecfc1314-a0cb-4bac-a35c-d2175f1c7197"
-					(reference "ANT1")
+					(reference "ANT_S1")
 					(unit 1)
 				)
@@
 		(on_board yes)
 		(dnp no)
-		(fields_autoplaced yes)
-		(property "Reference" "FB4"
+		(property "Reference" "FB_R1"
 			(at 236.1819 30.48 90)
 			(effects
@@
 			(project "RicardoTemplate"
 				(path "/7db990e4-92e1-4f99-b4d2-435bbec1ba83/ecfc1314-a0cb-4bac-a35c-d2175f1c7197"
-					(reference "FB4")
+					(reference "FB_R1")
 					(unit 1)
 				)
