File: RicardoTemplate.kicad_sch (KiCad schematic)
At the start: 39 parts, among them J1 RBUS, U1 ESP32-S3, Y1 R940000171

Commit message: Alpha revision
Bulk of routing, layout and etc... is done, design needs to be refined, via stitched and reviewed.
Parts:
- added JTAG1: JTAG, Connector_PinHeader_2.54mm:PinHeader_1x04_P2.54mm_Vertical, symbol Connector_Generic:Conn_01x04
- added TP24, TP25: TestPoint, TestPoint:TestPoint_Pad_D1.0mm, symbol Connector:TestPoint
- added UART1: UART, Connector_PinHeader_2.54mm:PinHeader_1x04_P2.54mm_Vertical, symbol Connector_Generic:Conn_01x04
- U1: footprint iclr:QFN40P700X700X90-57N -> footprints:QFN40P700X700X90-57N
Connections:
- net +3V3: now also UART1.4 (Pin_4)
- net ANT_SEL: now also U1.14 (GPIO9/ADC1_CH8)
- net CAN_RX: now also TP10.1, U1.23 (GPIO17/ADC2_CH6/DAC_2)
- net CAN_TX: now also TP9.1, U1.24 (GPIO18/ADC2_CH7/DAC_1)
- net CHL: now also U1.17 (GPIO12/ADC2_CH1)
- net CPS: now also U1.19 (GPIO14/ADC2_CH3)
- net CRX: now also U1.16 (GPIO11/ADC2_CH0)
- net CSD: now also U1.15 (GPIO10/ADC1_CH9)
- net CTX: now also U1.18 (GPIO13/ADC2_CH2)
- net GND: now also UART1.1 (Pin_1)
- net RXD: now also UART1.3 (Pin_3); no longer TP10.1
- net TXD: now also UART1.2 (Pin_2); no longer TP9.1
- net DIO1: now reaches U1.11 (GPIO6/ADC1_CH5)
- net SX_BUSY: now reaches U1.12 (GPIO7/ADC1_CH6)
- net RF_RST: now reaches U1.13 (GPIO8/ADC1_CH7)
- net at U1.44 (MTCK/JTAG/GPIO39): now also JTAG1.4 (Pin_4)
- net at U1.45 (MTDO/JTAG/GPIO40): now also JTAG1.3 (Pin_3)
- net at U1.47 (MTDI/JTAG/GPIO41): now also JTAG1.2 (Pin_2)
- net at U1.48 (MTMS/JTAG/GPIO42): now also JTAG1.1 (Pin_1)
- net CLK renamed SCK

Commit message: Minor improvements
Parts:
- removed JTAG1: JTAG, Connector_PinHeader_2.54mm:PinHeader_1x04_P2.54mm_Vertical, symbol Connector_Generic:Conn_01x04
- removed TP24, TP25: TestPoint, TestPoint:TestPoint_Pad_D1.0mm, symbol Connector:TestPoint
- renumbered TP10 to CANRX1, TP9 to CANTX1
