File: power.kicad_sch (KiCad schematic)
At the start: 20 parts, among them U3 LM66200DRLR, U4 MAX77827AEFD+T, U5 SC4215ASTRT

Commit message: Alpha revision
Bulk of routing, layout and etc... is done, design needs to be refined, via stitched and reviewed.
Parts:
- added BOOTJUMPER3: Conn_01x02_Male, Connector_PinHeader_2.54mm:PinHeader_1x02_P2.54mm_Vertical, symbol Connector:Conn_01x02_Male
- added FB1: FerriteBead_Small, Inductor_SMD:L_0603_1608Metric, symbol Device:FerriteBead_Small
- U3: footprint iclr:SOTFL50P160X60-8N -> footprints:SOTFL50P160X60-8N
- U4: footprint iclr:CONV_MAX77827AEFD+T -> footprints:CONV_MAX77827AEFD+T
- U5: footprint iclr:SOIC127P599X175-9N -> footprints:SOIC127P599X175-9N
Connections:
- net +3V3: now also FB1.2; no longer C26.2, C27.2, R16.1, U5.6 (VOUT)
- new net: BOOTJUMPER3.2 (Pin_2), C26.2, C27.2, R16.1, U5.6 (VOUT)
- new net: BOOTJUMPER3.1 (Pin_1), FB1.1
Other:
- moved on the sheet: C20, C21, C22, C23, C24, C25, C26, C27, L3, R15, R16, R17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

Commit message: Minor improvements
Parts:
- renumbered FB1 to FB_P1, BOOTJUMPER3 to POWER_MAIN1
Connections:
- net VBUS: no longer C23.1, C24.1, C25.1, TP8.1, U4.11 (OUT), U4.13 (OUTS), U5.2 (EN), U5.3 (VIN)
- new net BBOUT: C23.1, C24.1, C25.1, TP8.1, U4.11 (OUT), U4.13 (OUTS), U5.2 (EN), U5.3 (VIN)
Changed lines of the file:
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@@
 	)
 	(junction
-		(at 118.11 76.2)
-		(diameter 0)
-		(color 0 0 0 0)
-	)
-	(junction
 		(at 172.72 76.2)
 		(diameter 0)
@@
 	(wire
 		(pts
-			(xy 114.3 76.2) (xy 118.11 76.2)
-		)
-		(stroke
-			(width 0)
-			(type default)
-		)
-	)
-	(wire
-		(pts
 			(xy 45.72 88.9) (xy 55.88 88.9)
 		)
@@
 	(wire
 		(pts
-			(xy 118.11 76.2) (xy 123.19 76.2)
+			(xy 114.3 76.2) (xy 123.19 76.2)
 		)
 		(stroke
@@
 	)
 	(symbol
-		(lib_name "VBUS_1")
-		(lib_id "power:VBUS")
-		(at 118.11 76.2 0)
-		(unit 1)
-		(exclude_from_sim no)
-		(in_bom yes)
-		(on_board yes)
-		(dnp no)
-		(fields_autoplaced yes)
-		(property "Reference" "#PWR073"
-			(at 118.11 80.01 0)
-			(effects
-				(font
-					(size 1.27 1.27)
-				)
-				(hide yes)
-			)
-		)
-		(property "Value" "VBUS"
-			(at 118.11 71.12 0)
-			(effects
-				(font
-					(size 1.27 1.27)
-				)
-			)
-		)
-		(property "Footprint" ""
-			(at 118.11 76.2 0)
-			(effects
-				(font
-					(size 1.27 1.27)
-				)
-				(hide yes)
-			)
-		)
-		(property "Datasheet" ""
-			(at 118.11 76.2 0)
-			(effects
-				(font
-					(size 1.27 1.27)
-				)
-				(hide yes)
-			)
-		)
-		(property "Description" "Power symbol creates a global label with name \"VBUS\""
-			(at 118.11 76.2 0)
-			(effects
-				(font
-					(size 1.27 1.27)
-				)
-				(hide yes)
-			)
-		)
-		(pin "1"
-		)
-		(instances
-			(project ""
-				(path "/7db990e4-92e1-4f99-b4d2-435bbec1ba83/48a413b4-b7c2-44ac-971c-583c31b73475"
-					(reference "#PWR073")
-					(unit 1)
-				)
-			)
-		)
-	)
-	(symbol
 		(lib_id "power:GND")
 		(at 138.43 91.44 0)
@@
 		(on_board yes)
 		(dnp no)
-		(property "Reference" "BOOTJUMPER3"
+		(property "Reference" "POWER_MAIN1"
 			(at 186.69 66.04 90)
 			(effects
@@
 			(project "RicardoTemplate"
 				(path "/7db990e4-92e1-4f99-b4d2-435bbec1ba83/48a413b4-b7c2-44ac-971c-583c31b73475"
-					(reference "BOOTJUMPER3")
+					(reference "POWER_MAIN1")
 					(unit 1)
 				)
@@
 		(dnp no)
 		(fields_autoplaced yes)
-		(property "Reference" "FB1"
+		(property "Reference" "FB_P1"
 			(at 205.7019 69.85 90)
 			(effects
@@
 			(project "RicardoTemplate"
 				(path "/7db990e4-92e1-4f99-b4d2-435bbec1ba83/48a413b4-b7c2-44ac-971c-583c31b73475"
-					(reference "FB1")
+					(reference "FB_P1")
 					(unit 1)
 				)
